Commit message: Fixed tree branching

File: src/navigation/urdf/macros.xacro (robot description, xacro)
@@ -4,5 +4,4 @@
                params="default_antenna:=true
                        rockers_fixed:=true
-                       footprint_link:=true
                        link_prefix:=''
                        joint_prefix:=''
@@ -94,7 +93,4 @@
     </xacro:macro>
     <!-- LINKS -->
-    <xacro:if value="${footprint_link}">
-      <link name="${link_prefix}base_footprint"/>
-    </xacro:if>
     <link name="${link_prefix}base_link">
       <inertial>
@@ -158,11 +154,4 @@
     <link name="${link_prefix}imu_frame"/>
     <!-- JOINTS -->
-    <xacro:if value="${footprint_link}">
-      <joint name="${joint_prefix}base_joint" type="fixed">
-        <origin xyz="0 0 0.19783" rpy="0 0 0"/>
-        <parent link="${link_prefix}base_footprint"/>
-        <child link="${link_prefix}base_link"/>
-      </joint>
-    </xacro:if>
     <xacro:if value="${rockers_fixed}">
       <xacro:property name="rockers_joint_type" value="fixed"/>
@@ -263,5 +252,5 @@
     </joint>
   </xacro:macro>
-    <!-- Leo_sim -->
+  <!-- Leo_sim -->
   <xacro:macro name="leo_sim"
                params="default_antenna:=true
